File: schematics/esp32_fc.kicad_sch (KiCad schematic)
At the start: 18 parts, among them J5 Conn_01x02_Pin, J6 Conn_01x08_Socket, J7 USB_C_Receptacle_USB2.0_16P, SW1 SW_SPST, SW2 SW_SPST, U1 ESP32-WROOM-32D, U2 AP2112K-3.3TRG1, U3 CP2102N-Axx-xQFN20

Commit message: changed espfc schematic
Parts:
- added D10, D7, D8, D9: LED, LED_SMD:LED_0603_1608Metric, symbol Device:LED
- added J10, J11, J8, J9: Conn_01x02_Pin, Connector_JST:JST_XH_B2B-XH-A_1x02_P2.50mm_Vertical, symbol Connector:Conn_01x02_Pin
- added Q5, Q6, Q7, Q8: IRLML6244, Package_TO_SOT_SMD:SOT-23, symbol Transistor_FET:IRLML6244
- added R10, R11, R8, R9: 10K, Resistor_SMD:R_0603_1608Metric, symbol Device:R
Connections:
- net 3.7V: now also D10.1 (K), D7.1 (K), D8.1 (K), D9.1 (K), J10.1 (Pin_1), J11.1 (Pin_1), J8.1 (Pin_1), J9.1 (Pin_1)
- net GND: now also Q5.2 (S), Q6.2 (S), Q7.2 (S), Q8.2 (S), R10.2, R11.2, R8.2, R9.2
- new net: D8.2 (A), J9.2 (Pin_2), Q6.3 (D)
- new net: D10.2 (A), J11.2 (Pin_2), Q8.3 (D)
- new net: D9.2 (A), J10.2 (Pin_2), Q7.3 (D)
- new net: D7.2 (A), J8.2 (Pin_2), Q5.3 (D)
- new net GPIO: Q5.1 (G), Q6.1 (G), Q7.1 (G), Q8.1 (G), R10.1, R11.1, R8.1, R9.1
Other:
- removed sheet Motor Driver
- removed sheet Motor Driver1
- removed sheet Motor Driver2
- removed sheet Motor Driver3
- moved on the sheet: C1, C2, C3, C4, C5, D5, D6, J5, J6, J7, R5, R6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
